File: Single Key.kicad_sch (KiCad schematic)
At the start: 20 parts, among them SW1 SW_Push, SW10 SW_Push, SW11 SW_Push, SW12 SW_Push, SW13 SW_Push, SW14 SW_Push, SW15 SW_Push, SW16 SW_Push, SW17 SW_Push, SW18 SW_Push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

Commit message: new updates
Parts:
- added J1: Conn_01x05_Pin, Connector_PinHeader_2.54mm:PinHeader_1x05_P2.54mm_Vertical, symbol Connector:Conn_01x05_Pin
Connections:
- net ROW1: now also J1.1 (Pin_1)
- net ROW2: now also J1.2 (Pin_2)
- net ROW3: now also J1.3 (Pin_3)
- net ROW4: now also J1.4 (Pin_4)
- net ROW5: now also J1.5 (Pin_5)

Commit message: new updates
Parts:
- added J2: Conn_01x04_Pin, Connector_PinSocket_2.54mm:PinSocket_1x04_P2.54mm_Vertical, symbol Connector:Conn_01x04_Pin
Connections:
- net Col1: now also J2.1 (Pin_1)
- net Col2: now also J2.2 (Pin_2)
- net Col3: now also J2.3 (Pin_3)
- net Col4: now also J2.4 (Pin_4)
Changed lines of the file:
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@@
+	)
+	(junction
+		(at 179.07 40.64)
+		(diameter 0)
+		(color 0 0 0 0)
 	)
 	(junction
@@
 	)
 	(junction
+		(at 113.03 40.64)
+		(diameter 0)
+		(color 0 0 0 0)
+	)
+	(junction
+		(at 157.48 39.37)
+		(diameter 0)
+		(color 0 0 0 0)
+	)
+	(junction
 		(at 135.89 63.5)
 		(diameter 0)
@@
 	)
 	(junction
+		(at 135.89 40.64)
+		(diameter 0)
+		(color 0 0 0 0)
+	)
+	(junction
 		(at 119.38 95.25)
 		(diameter 0)
@@
 	(wire
 		(pts
-			(xy 179.07 35.56) (xy 179.07 49.53)
+			(xy 179.07 35.56) (xy 179.07 40.64)
 		)
 		(stroke
@@
 	(wire
 		(pts
+			(xy 146.05 39.37) (xy 157.48 39.37)
+		)
+		(stroke
+			(width 0)
+			(type default)
+		)
+	)
+	(wire
+		(pts
 			(xy 119.38 105.41) (xy 121.92 105.41)
 		)
@@
 	(wire
 		(pts
-			(xy 113.03 35.56) (xy 113.03 49.53)
+			(xy 113.03 35.56) (xy 113.03 40.64)
 		)
 		(stroke
@@
 	(wire
 		(pts
+			(xy 179.07 40.64) (xy 179.07 49.53)
+		)
+		(stroke
+			(width 0)
+			(type default)
+		)
+	)
+	(wire
+		(pts
 			(xy 119.38 91.44) (xy 121.92 91.44)
 		)
@@
 	(wire
 		(pts
+			(xy 146.05 24.13) (xy 146.05 39.37)
+		)
+		(stroke
+			(width 0)
+			(type default)
+		)
+	)
+	(wire
+		(pts
 			(xy 83.82 81.28) (xy 91.44 81.28)
 		)
@@
 	(wire
 		(pts
+			(xy 148.59 24.13) (xy 173.99 24.13)
+		)
+		(stroke
+			(width 0)
+			(type default)
+		)
+	)
+	(wire
+		(pts
+			(xy 143.51 40.64) (xy 135.89 40.64)
+		)
+		(stroke
+			(width 0)
+			(type default)
+		)
+	)
+	(wire
+		(pts
 			(xy 157.48 49.53) (xy 157.48 63.5)
 		)
@@
 	(wire
 		(pts
+			(xy 173.99 24.13) (xy 173.99 40.64)
+		)
+		(stroke
+			(width 0)
+			(type default)
+		)
+	)
+	(wire
+		(pts
 			(xy 83.82 109.22) (xy 92.71 109.22)
 		)
@@
 	(wire
 		(pts
-			(xy 157.48 35.56) (xy 157.48 49.53)
+			(xy 157.48 35.56) (xy 157.48 39.37)
+		)
+		(stroke
+			(width 0)
+			(type default)
+		)
+	)
+	(wire
+		(pts
+			(xy 143.51 24.13) (xy 143.51 40.64)
+		)
+		(stroke
+			(width 0)
+			(type default)
+		)
+	)
+	(wire
+		(pts
+			(xy 140.97 24.13) (xy 119.38 24.13)
+		)
+		(stroke
+			(width 0)
+			(type default)
+		)
+	)
+	(wire
+		(pts
+			(xy 135.89 40.64) (xy 135.89 49.53)
 		)
 		(stroke
@@
 	(wire
 		(pts
+			(xy 157.48 39.37) (xy 157.48 49.53)
+		)
+		(stroke
+			(width 0)
+			(type default)
+		)
+	)
+	(wire
+		(pts
 			(xy 163.83 91.44) (xy 163.83 95.25)
 		)
@@
 	(wire
 		(pts
-			(xy 135.89 35.56) (xy 135.89 49.53)
+			(xy 135.89 35.56) (xy 135.89 40.64)
 		)
 		(stroke
@@
 	(wire
 		(pts
+			(xy 113.03 40.64) (xy 113.03 49.53)
+		)
+		(stroke
+			(width 0)
+			(type default)
+		)
+	)
+	(wire
+		(pts
 			(xy 140.97 49.53) (xy 140.97 53.34)
 		)
@@
 	(wire
 		(pts
+			(xy 119.38 40.64) (xy 113.03 40.64)
+		)
+		(stroke
+			(width 0)
+			(type default)
+		)
+	)
+	(wire
+		(pts
 			(xy 135.89 49.53) (xy 132.08 49.53)
+		)
+		(stroke
+			(width 0)
+			(type default)
+		)
+	)
+	(wire
+		(pts
+			(xy 119.38 24.13) (xy 119.38 40.64)
+		)
+		(stroke
+			(width 0)
+			(type default)
+		)
+	)
+	(wire
+		(pts
+			(xy 173.99 40.64) (xy 179.07 40.64)
 		)
 		(stroke
@@
 					(unit 1)
 				)
+			)
+		)
+	)
+	(symbol
+		(lib_id "Connector:Conn_01x04_Pin")
+		(at 143.51 19.05 90)
+		(mirror x)
+		(unit 1)
+		(exclude_from_sim no)
+		(in_bom yes)
+		(on_board yes)
+		(dnp no)
+		(property "Reference" "J2"
+			(at 144.78 13.97 90)
+			(effects
+				(font
+					(size 1.27 1.27)
+				)
+			)
+		)
+		(property "Value" "Conn_01x04_Pin"
+			(at 144.78 16.51 90)
+			(effects
+				(font
+					(size 1.27 1.27)
+				)
+			)
+		)
+		(property "Footprint" "Connector_PinSocket_2.54mm:PinSocket_1x04_P2.54mm_Vertical"
+			(at 143.51 19.05 0)
+			(effects
+				(font
+					(size 1.27 1.27)
+				)
+				(hide yes)
+			)
+		)
+		(property "Datasheet" "~"
+			(at 143.51 19.05 0)
+			(effects
+				(font
+					(size 1.27 1.27)
+				)
+				(hide yes)
+			)
+		)
+		(property "Description" "Generic connector, single row, 01x04, script generated"
+			(at 143.51 19.05 0)
+			(effects
+				(font
+					(size 1.27 1.27)
+				)
+				(hide yes)
+			)
+		)
+		(pin "1"
+		)
+		(pin "3"
+		)
+		(pin "4"
+		)
+		(pin "2"
+		)
+		(instances
+			(project ""
+				(path "/23b3dbb6-255b-4abd-a420-3ae1e40d4999"
+					(reference "J2")
+					(unit 1)
+				)
