File: Single Key.kicad_pcb (KiCad board)
At the start: 2 copper layers, 4 parts, among them J1 4pin Molex Male, J2 2Pin Header - Key, J3 2Pin Header - Solenoid

Commit message: new updates
Parts:
- removed D1: D, Diode_THT:D_A-405_P10.16mm_Horizontal
- removed J2: 2Pin Header - Key, Connector_PinHeader_2.54mm:PinHeader_1x02_P2.54mm_Vertical
- removed J3: 2Pin Header - Solenoid, Connector_PinHeader_2.54mm:PinHeader_1x02_P2.54mm_Vertical
- added SW1: SW_Push, Button_Switch_THT:SW_PUSH_6mm, F.Cu at (119.4, 66.5)
- added SW10: SW_Push, Button_Switch_THT:SW_PUSH_6mm, F.Cu at (144.6, 75.0)
- added SW11: SW_Push, Button_Switch_THT:SW_PUSH_6mm, F.Cu at (144.6, 83.6)
- added SW12: SW_Push, Button_Switch_THT:SW_PUSH_6mm, F.Cu at (144.6, 92.2)
- added SW13: SW_Push, Button_Switch_THT:SW_PUSH_6mm, F.Cu at (155.1, 66.5)
- added SW14: SW_Push, Button_Switch_THT:SW_PUSH_6mm, F.Cu at (155.1, 75.0)
- added SW15: SW_Push, Button_Switch_THT:SW_PUSH_6mm, F.Cu at (155.1, 83.6)
- added SW16: SW_Push, Button_Switch_THT:SW_PUSH_6mm, F.Cu at (155.1, 92.2)
- added SW17: SW_Push, Button_Switch_THT:SW_PUSH_6mm, F.Cu at (165.7, 66.5)
- added SW18: SW_Push, Button_Switch_THT:SW_PUSH_6mm, F.Cu at (165.7, 75.0)
- added SW19: SW_Push, Button_Switch_THT:SW_PUSH_6mm, F.Cu at (165.7, 83.6)
- added SW2: SW_Push, Button_Switch_THT:SW_PUSH_6mm, F.Cu at (119.4, 75.0)
- added SW20: SW_Push, Button_Switch_THT:SW_PUSH_6mm, F.Cu at (165.7, 92.2)
- added SW3: SW_Push, Button_Switch_THT:SW_PUSH_6mm, F.Cu at (119.4, 83.5)
- added SW4: SW_Push, Button_Switch_THT:SW_PUSH_6mm, F.Cu at (119.4, 92.1)
- added SW5: SW_Push, Button_Switch_THT:SW_PUSH_6mm, F.Cu at (132.1, 66.4)
- added SW6: SW_Push, Button_Switch_THT:SW_PUSH_6mm, F.Cu at (132.1, 75.0)
- added SW7: SW_Push, Button_Switch_THT:SW_PUSH_6mm, F.Cu at (132.1, 83.5)
- added SW8: SW_Push, Button_Switch_THT:SW_PUSH_6mm, F.Cu at (132.1, 92.0)
- added SW9: SW_Push, Button_Switch_THT:SW_PUSH_6mm, F.Cu at (144.6, 66.5)
- J1: value 4pin Molex Male -> Conn_01x05_Pin; footprint Connector_Molex:Molex_SPOX_5267-04A_1x04_P2.50mm_Vertical -> Connector_PinHeader_2.54mm:PinHeader_1x05_P2.54mm_Vertical
- moved J1 24.3 mm to (97.2, 74.2)
Connections:
- J1 pad 1: Net-(D1-K) -> ROW1
- J1 pad 2: Net-(J1-Pin_2) -> ROW2
- J1 pad 3: Net-(J1-Pin_3) -> ROW3
- J1 pad 4: Net-(J1-Pin_4) -> ROW4

Commit message: new updates
Parts:
- added J2: Conn_01x04_Pin, Connector_PinSocket_2.54mm:PinSocket_1x04_P2.54mm_Vertical, F.Cu at (185.4, 75.6)
- moved J1 62.4 mm to (149.2, 108.6), turned to 90 degrees
- moved SW20 7.55 mm to (171.4, 97.1)
- moved SW19 6.49 mm to (171.4, 86.7)
- moved SW17 6.33 mm to (171.4, 63.8)
- moved SW16 5.75 mm to (158.0, 97.1)
- moved SW18 5.73 mm to (171.4, 75.2)
- moved SW8 5.05 mm to (132.0, 97.1)
- moved SW4 5.00 mm to (119.4, 97.1)
- moved SW12 4.95 mm to (144.7, 97.1)
- moved SW15 4.24 mm to (158.0, 86.7)
- moved SW13 4.00 mm to (158.0, 63.8)
- moved SW3 3.10 mm to (119.4, 86.7)
- moved SW11 3.05 mm to (144.7, 86.7)
- moved SW14 2.94 mm to (158.0, 75.0)
- moved SW7 2.86 mm to (132.1, 86.4)
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Routing:
- net ROW1: track 0.00 -> 79.7 mm
- net ROW2: track 0.00 -> 64.8 mm
- net Col4: track 0.00 -> 21.5 mm
- net ROW5: track 0.00 -> 21.3 mm
- net Col3: track 0.00 -> 14.1 mm
- net ROW4: track 0.00 -> 13.4 mm
- net ROW3: track 0.00 -> 12.8 mm
- net Col1: track 0.00 -> 11.5 mm
- net Col2: track 0.00 -> 8.23 mm

Commit message: new updates
Parts:
- moved J1 43.4 mm to (185.7, 85.1), turned to 0 degrees
- moved SW3 6.52 mm to (112.9, 86.1)
- moved SW1 6.50 mm to (112.9, 63.8)
- moved SW2 6.50 mm to (112.9, 75.0)
- moved SW4 6.50 mm to (112.9, 97.1)
- moved SW7 5.06 mm to (127.0, 86.1)
- moved SW6 5.02 mm to (127.0, 75.1)
- moved SW8 5.00 mm to (127.0, 97.1)
- moved SW5 5.00 mm to (127.1, 63.8)
- moved J2 4.71 mm to (185.7, 70.9)
- moved SW11 3.72 mm to (141.0, 86.1)
- moved SW9 3.69 mm to (141.0, 63.9)
- moved SW12 3.68 mm to (141.0, 97.2)
- moved SW10 3.53 mm to (141.0, 75.2)
- moved SW15 2.64 mm to (155.4, 86.1)
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Routing:
- net ROW3: track 12.8 -> 119.1 mm
- net ROW1: track 79.7 -> 169.5 mm
- net ROW4: track 13.4 -> 99.9 mm
- net ROW2: track 64.8 -> 145.8 mm
- net ROW5: track 21.3 -> 75.0 mm
- net Col4: track 21.5 -> 60.1 mm
- net Col3: track 14.1 -> 52.0 mm
- net Col2: track 8.23 -> 43.0 mm
- net Col1: track 11.5 -> 41.8 mm

Commit message: new updates
Routing:
- net ROW1: track 169.5 -> 167.5 mm
- net ROW2: track 145.8 -> 144.2 mm
Other:
- board text added: "Matrix Keyboard"
- board text added: "© JR Payos March 2025"
Changed lines of the file:
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@@
 		(pad "1" thru_hole rect
 			(at 0 0)
-			(size 1.7 1.7)
-			(drill 1)
+			(size 1.8 1.8)
+			(drill 0.8)
 			(layers "*.Cu" "*.Mask")
 			(remove_unused_layers no)
@@
 		(pad "2" thru_hole oval
 			(at 0 2.54)
-			(size 1.7 1.7)
-			(drill 1)
+			(size 1.8 1.8)
+			(drill 0.8)
 			(layers "*.Cu" "*.Mask")
 			(remove_unused_layers no)
@@
 		(pad "3" thru_hole oval
 			(at 0 5.08)
-			(size 1.7 1.7)
-			(drill 1)
+			(size 1.8 1.8)
+			(drill 0.8)
 			(layers "*.Cu" "*.Mask")
 			(remove_unused_layers no)
@@
 		(pad "4" thru_hole oval
 			(at 0 7.62)
-			(size 1.7 1.7)
-			(drill 1)
+			(size 1.8 1.8)
+			(drill 0.8)
 			(layers "*.Cu" "*.Mask")
 			(remove_unused_layers no)
@@
 		(pad "5" thru_hole oval
 			(at 0 10.16)
-			(size 1.7 1.7)
-			(drill 1)
+			(size 1.8 1.8)
+			(drill 0.8)
 			(layers "*.Cu" "*.Mask")
 			(remove_unused_layers no)
@@
 		(net 2)
 	)
+	(gr_text "© JR Payos\nMarch 2025"
+		(at 193.04 80.264 90)
+		(layer "F.Cu")
+		(effects
+			(font
+				(size 1.5 1.5)
+				(thickness 0.3)
+				(bold yes)
+			)
+			(justify left bottom)
+		)
+	)
+	(gr_text "Matrix Keyboard"
+		(at 111.506 111.506 0)
+		(layer "F.Cu")
+		(effects
+			(font
+				(size 1.5 1.5)
+				(thickness 0.3)
+				(bold yes)
+			)
+			(justify left bottom)
+		)
+	)
 	(segment
 		(start 172.72 95.25)
@@
 	)
 	(segment
+		(start 129.032 105.156)
+		(end 132.334 108.458)
+		(width 1.016)
+		(layer "F.Cu")
+		(net 2)
+	)
+	(segment
 		(start 119.182 86.36)
 		(end 118.182 86.36)
@@
 	)
 	(segment
-		(start 119.182 64.008)
-		(end 119.4 63.79)
+		(start 112.88 97.1)
+		(end 116.15 100.37)
 		(width 1.016)
 		(layer "F.Cu")
@@
 	)
 	(segment
-		(start 119.4 86.142)
-		(end 119.182 86.36)
+		(start 119.182 64.008)
+		(end 119.4 63.79)
 		(width 1.016)
 		(layer "F.Cu")
@@
 	)
 	(segment
-		(start 195.072 106.426)
-		(end 195.072 89.916)
+		(start 119.4 86.142)
+		(end 119.182 86.36)
 		(width 1.016)
 		(layer "F.Cu")
@@
 	)
 	(segment
-		(start 149.225 108.585)
+		(start 149.098 108.458)
 		(end 152.4 111.76)
 		(width 1.016)
@@
 	)
 	(segment
-		(start 118.563 108.585)
-		(end 149.225 108.585)
-		(width 1.016)
-		(layer "F.Cu")
-		(net 2)
-	)
-	(segment
 		(start 116.15 96.012)
 		(end 116.15 88.392)
@@
 	)
 	(segment
-		(start 189.738 111.76)
-		(end 195.072 106.426)
+		(start 118.618 105.156)
+		(end 129.032 105.156)
 		(width 1.016)
 		(layer "F.Cu")
@@
 	)
 	(segment
-		(start 152.4 111.76)
-		(end 189.738 111.76)
+		(start 190.246 85.09)
+		(end 185.674 85.09)
 		(width 1.016)
 		(layer "F.Cu")
@@
 	)
 	(segment
-		(start 116.15 106.172)
-		(end 118.563 108.585)
+		(start 116.15 88.392)
+		(end 116.15 76.708)
 		(width 1.016)
 		(layer "F.Cu")
@@
 	)
 	(segment
-		(start 116.15 88.392)
-		(end 116.15 76.708)
+		(start 195.072 106.426)
+		(end 195.072 89.916)
 		(width 1.016)
 		(layer "F.Cu")
@@
 	)
 	(segment
-		(start 112.88 97.1)
-		(end 116.15 100.37)
+		(start 119.4 75)
+		(end 119.216 75.184)
 		(width 1.016)
 		(layer "F.Cu")
@@
 	)
 	(segment
-		(start 119.4 75)
-		(end 119.216 75.184)
+		(start 152.4 111.76)
+		(end 189.738 111.76)
 		(width 1.016)
 		(layer "F.Cu")
@@
 	)
 	(segment
-		(start 116.15 100.37)
-		(end 116.15 106.172)
+		(start 116.15 102.688)
+		(end 118.618 105.156)
 		(width 1.016)
 		(layer "F.Cu")
@@
 	)
 	(segment
-		(start 190.246 85.09)
-		(end 185.674 85.09)
+		(start 132.334 108.458)
+		(end 149.098 108.458)
+		(width 1.016)
+		(layer "F.Cu")
+		(net 2)
+	)
+	(segment
+		(start 195.072 89.916)
+		(end 190.246 85.09)
+		(width 1.016)
+		(layer "F.Cu")
+		(net 2)
+	)
+	(segment
+		(start 116.15 100.37)
+		(end 116.15 102.688)
 		(width 1.016)
 		(layer "F.Cu")
@@
 	)
 	(segment
-		(start 195.072 89.916)
-		(end 190.246 85.09)
+		(start 189.738 111.76)
+		(end 195.072 106.426)
 		(width 1.016)
 		(layer "F.Cu")
@@
 	)
 	(segment
-		(start 130.028 104.882)
-		(end 130.028 100.06)
-		(width 1.016)
-		(layer "F.Cu")
-		(net 5)
-	)
-	(segment
 		(start 130.556 87.376)
 		(end 131.862 86.07)
@@
 	)
 	(segment
-		(start 131.318 106.172)
-		(end 130.028 104.882)
-		(width 1.016)
-		(layer "F.Cu")
-		(net 5)
-	)
-	(segment
-		(start 154.559 109.728)
-		(end 151.003 106.172)
-		(width 1.016)
-		(layer "F.Cu")
-		(net 5)
-	)
-	(segment
-		(start 151.003 106.172)
-		(end 131.318 106.172)
-		(width 1.016)
-		(layer "F.Cu")
-		(net 5)
-	)
-	(segment
 		(start 130.556 95.504)
 		(end 130.556 89.046)
@@
 	)
 	(segment
+		(start 192.786 104.14)
+		(end 187.198 109.728)
+		(width 1.016)
+		(layer "F.Cu")
+		(net 5)
+	)
+	(segment
 		(start 132.679 75.093)
 		(end 133.532 75.093)
@@
 	)
 	(segment
-		(start 192.786 104.14)
-		(end 187.198 109.728)
+		(start 134.112 106.172)
+		(end 130.028 102.088)
 		(width 1.016)
 		(layer "F.Cu")
@@
 	)
 	(segment
-		(start 185.674 87.63)
-		(end 188.976 87.63)
+		(start 151.003 106.172)
+		(end 134.112 106.172)
 		(width 1.016)
 		(layer "F.Cu")
@@
 	)
 	(segment
-		(start 188.976 87.63)
-		(end 192.786 91.44)
+		(start 130.028 100.06)
+		(end 127.032 97.064)
 		(width 1.016)
 		(layer "F.Cu")
@@
 	)
 	(segment
+		(start 185.674 87.63)
+		(end 188.976 87.63)
+		(width 1.016)
+		(layer "F.Cu")
+		(net 5)
+	)
+	(segment
 		(start 130.556 65.024)
 		(end 131.79 63.79)
@@
 	)
 	(segment
+		(start 192.786 91.44)
+		(end 192.786 104.14)
+		(width 1.016)
+		(layer "F.Cu")
+		(net 5)
+	)
+	(segment
+		(start 154.559 109.728)
+		(end 151.003 106.172)
+		(width 1.016)
+		(layer "F.Cu")
+		(net 5)
+	)
+	(segment
 		(start 130.556 77.216)
 		(end 132.679 75.093)
@@
 	)
 	(segment
-		(start 130.028 100.06)
-		(end 127.032 97.064)
+		(start 130.028 102.088)
+		(end 130.028 100.06)
 		(width 1.016)
 		(layer "F.Cu")
@@
 	)
 	(segment
-		(start 130.556 96.012)
-		(end 130.556 95.504)
+		(start 188.976 87.63)
+		(end 192.786 91.44)
 		(width 1.016)
 		(layer "F.Cu")
@@
 	)
 	(segment
-		(start 192.786 91.44)
-		(end 192.786 104.14)
+		(start 130.556 96.012)
+		(end 130.556 95.504)
 		(width 1.016)
 		(layer "F.Cu")

Commit message: new update
Other:
- board text added: "4x5 Matrix Keyboard"
- board text removed: "Matrix Keyboard"
Changed lines of the file:
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@@
 		)
 	)
-	(gr_text "Matrix Keyboard"
-		(at 111.506 111.506 0)
+	(gr_text "4x5 Matrix Keyboard"
+		(at 111.506 112.014 0)
 		(layer "F.Cu")
 		(effects
